Commit message: fix!: make model A lidar mounts fixed
Keep sensor geometry in the model and restore a level front lidar.
Verify fixed mounts and ignored overrides with regression tests.

BREAKING CHANGE: front_top_lidar_mount and back_bottom_lidar_mount
are no longer configurable Xacro arguments.

File: urdf/robot_forki3_a.xacro (robot description, xacro)
@@ -53,8 +53,4 @@
   <xacro:arg name="front_top_lidar_use_c_mesh"         default="True"/>
   <xacro:arg name="front_top_lidar_c_mesh_use_low_res" default="True"/>
-  <!-- Positive pitch tilts the lidar 30 degrees toward the ground on the robot's +X side. -->
-  <!-- Restore the commented level pose to compare ground coverage with the original mount. -->
-  <!-- <xacro:arg name="front_top_lidar_mount" default="-0.07647355 0 1.786 0 0 0"/> -->
-  <xacro:arg name="front_top_lidar_mount" default="-0.07647355 0 1.786 0 0.5235987755982988 0"/>
   <xacro:property name="front_top_lidar_use_visual"         value="$(arg front_top_lidar_use_visual)"/>
   <xacro:property name="front_top_lidar_use_collision"      value="$(arg front_top_lidar_use_collision)"/>
@@ -65,9 +61,5 @@
   <xacro:property name="front_top_lidar_use_c_mesh"         value="$(arg front_top_lidar_use_c_mesh)"/>
   <xacro:property name="front_top_lidar_c_mesh_use_low_res" value="$(arg front_top_lidar_c_mesh_use_low_res)"/>
-  <xacro:property name="front_top_lidar_mount"              value="$(arg front_top_lidar_mount)"/>
-  <xacro:property name="front_top_lidar_mount_seq"   value="${front_top_lidar_mount.split()}"/>
-  <xacro:if value="${len(front_top_lidar_mount_seq) != 6}">
-    ${xacro.fatal("xacro arg front_top_lidar_mount must have 6 elements: 'x y z roll pitch yaw'")}
-  </xacro:if>
+  <xacro:property name="front_top_lidar_mount" value="-0.07647355 0 1.786 0 0 0"/>
   <xacro:property name="front_top_lidar_sim_cfg"            value="${sim_cfg.get('front_top_lidar', dict())}"/>
   <!--
@@ -130,5 +122,4 @@
   <!-- Use the optimized collision mesh by default. -->
   <xacro:arg name="back_bottom_lidar_use_c_mesh"         default="True"/>
-  <xacro:arg name="back_bottom_lidar_mount" default="-0.692435 0 0.019941 0 0 3.141592653589793"/>
   <xacro:property name="back_bottom_lidar_use_visual"    value="$(arg back_bottom_lidar_use_visual)"/>
   <xacro:property name="back_bottom_lidar_use_collision" value="$(arg back_bottom_lidar_use_collision)"/>
@@ -137,5 +128,5 @@
   <xacro:property name="back_bottom_lidar_color"         value="$(arg back_bottom_lidar_color)"/>
   <xacro:property name="back_bottom_lidar_use_c_mesh"    value="$(arg back_bottom_lidar_use_c_mesh)"/>
-  <xacro:property name="back_bottom_lidar_mount"         value="$(arg back_bottom_lidar_mount)"/>
+  <xacro:property name="back_bottom_lidar_mount" value="-0.692435 0 0.019941 0 0 3.141592653589793"/>
   <xacro:property name="back_bottom_lidar_sim_cfg" value="${sim_cfg.get('back_bottom_lidar', dict())}"/>
   <xacro:set_props_plugin_lidar_2d prop_prefix="back_bottom_lidar_sim"
